File: can.kicad_sch (KiCad schematic)
At the start: 0 parts

Commit message: 回路図ほぼ完成 MOSFETのゲート抵抗の決め方よくわかんないです助けて
Parts:
- added C24: 100n, symbol Device:C
- added U3: SN65HVD230DR, digikey-footprints:SOIC-8_W3.9mm, symbol dk_Interface-Drivers-Receivers-Transceivers:SN65HVD230DR
Connections:
- new net +3V3: C24.2, U3.3 (VCC)
- new net CANH: U3.7 (CANH)
- new net CANL: U3.6 (CANL)
- new net CAN_RX: U3.4 (R)
- new net CAN_TX: U3.1 (D)
- new net GND: C24.1, U3.2 (GND), U3.8 (RS)
- no-connect marks 0 -> 1
Changed lines of the file:
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@@
 (kicad_sch (version 20230121) (generator eeschema)
   (paper "A4")
+  (junction (at 113.03 99.06) (diameter 0) (color 0 0 0 0)
+  )
+  (junction (at 123.19 99.06) (diameter 0) (color 0 0 0 0)
+  )
+  (junction (at 123.19 78.74) (diameter 0) (color 0 0 0 0)
+  )
+  (no_connect (at 130.81 88.9))
+  (wire (pts (xy 113.03 78.74) (xy 123.19 78.74))
+    (stroke (width 0) (type default))
+  )
+  (wire (pts (xy 113.03 99.06) (xy 123.19 99.06))
+    (stroke (width 0) (type default))
+  )
+  (wire (pts (xy 102.87 99.06) (xy 113.03 99.06))
+    (stroke (width 0) (type default))
+  )
+  (wire (pts (xy 113.03 91.44) (xy 113.03 99.06))
+    (stroke (width 0) (type default))
+  )
+  (wire (pts (xy 105.41 78.74) (xy 102.87 78.74))
+    (stroke (width 0) (type default))
+  )
+  (wire (pts (xy 102.87 78.74) (xy 102.87 99.06))
+    (stroke (width 0) (type default))
+  )
+  (hierarchical_label "CANL" (shape bidirectional) (at 113.03 86.36 180) (fields_autoplaced)
+    (effects (font (size 1.27 1.27)) (justify right))
+  )
+  (hierarchical_label "CAN_RX" (shape input) (at 130.81 86.36 0) (fields_autoplaced)
+    (effects (font (size 1.27 1.27)) (justify left))
+  )
+  (hierarchical_label "CANH" (shape bidirectional) (at 113.03 88.9 180) (fields_autoplaced)
+    (effects (font (size 1.27 1.27)) (justify right))
+  )
+  (hierarchical_label "CAN_TX" (shape output) (at 113.03 83.82 180) (fields_autoplaced)
+    (effects (font (size 1.27 1.27)) (justify right))
+  )
+  (symbol (lib_id "power:GND") (at 123.19 99.06 0) (unit 1)
+    (in_bom yes) (on_board yes) (dnp no) (fields_autoplaced)
+    (property "Reference" "#PWR038" (at 123.19 105.41 0)
+      (effects (font (size 1.27 1.27)) hide)
+    )
+    (property "Value" "GND" (at 123.19 104.14 0)
+      (effects (font (size 1.27 1.27)))
+    )
+    (property "Footprint" "" (at 123.19 99.06 0)
+      (effects (font (size 1.27 1.27)) hide)
+    )
+    (property "Datasheet" "" (at 123.19 99.06 0)
+      (effects (font (size 1.27 1.27)) hide)
+    )
+    (pin "1")
+    (instances
+      (project "blmd_hardware"
+        (path "/181c0b55-802a-4742-8349-1028710992a0/9e673ea1-d5ae-4157-89d9-c50410c687a1"
+          (reference "#PWR038") (unit 1)
+        )
+      )
+    )
+  )
+  (symbol (lib_id "dk_Interface-Drivers-Receivers-Transceivers:SN65HVD230DR") (at 120.65 81.28 0) (unit 1)
+    (in_bom yes) (on_board yes) (dnp no) (fields_autoplaced)
+    (property "Reference" "U3" (at 125.3841 76.2 0)
+      (effects (font (size 1.524 1.524)) (justify left))
+    )
+    (property "Value" "SN65HVD230DR" (at 125.3841 78.74 0)
+      (effects (font (size 1.524 1.524)) (justify left))
+    )
+    (property "Footprint" "digikey-footprints:SOIC-8_W3.9mm" (at 125.73 76.2 0)
+      (effects (font (size 1.524 1.524)) (justify left) hide)
+    )
+    (property "Datasheet" "http://www.ti.com/general/docs/suppproductinfo.tsp?distId=10&gotoUrl=http%3A%2F%2Fwww.ti.com%2Flit%2Fgpn%2Fsn65hvd230" (at 125.73 73.66 0)
+      (effects (font (size 1.524 1.524)) (justify left) hide)
+    )
+    (property "Digi-Key_PN" "296-11654-1-ND" (at 125.73 71.12 0)
+      (effects (font (size 1.524 1.524)) (justify left) hide)
+    )
+    (property "MPN" "SN65HVD230DR" (at 125.73 68.58 0)
+      (effects (font (size 1.524 1.524)) (justify left) hide)
+    )
+    (property "Category" "Integrated Circuits (ICs)" (at 125.73 66.04 0)
+      (effects (font (size 1.524 1.524)) (justify left) hide)
+    )
+    (property "Family" "Interface - Drivers, Receivers, Transceivers" (at 125.73 63.5 0)
+      (effects (font (size 1.524 1.524)) (justify left) hide)
+    )
+    (property "DK_Datasheet_Link" "http://www.ti.com/general/docs/suppproductinfo.tsp?distId=10&gotoUrl=http%3A%2F%2Fwww.ti.com%2Flit%2Fgpn%2Fsn65hvd230" (at 125.73 60.96 0)
+      (effects (font (size 1.524 1.524)) (justify left) hide)
+    )
+    (property "DK_Detail_Page" "/product-detail/en/texas-instruments/SN65HVD230DR/296-11654-1-ND/404366" (at 125.73 58.42 0)
+      (effects (font (size 1.524 1.524)) (justify left) hide)
+    )
+    (property "Description" "IC TXRX CAN 1MBPS 3.3V 8SOIC" (at 125.73 55.88 0)
+      (effects (font (size 1.524 1.524)) (justify left) hide)
+    )
+    (property "Manufacturer" "Texas Instruments" (at 125.73 53.34 0)
+      (effects (font (size 1.524 1.524)) (justify left) hide)
+    )
+    (property "Status" "Active" (at 125.73 50.8 0)
+      (effects (font (size 1.524 1.524)) (justify left) hide)
+    )
+    (pin "8")
+    (pin "6")
+    (pin "1")
+    (pin "5")
+    (pin "2")
+    (pin "3")
+    (pin "4")
+    (pin "7")
+    (instances
+      (project "blmd_hardware"
+        (path "/181c0b55-802a-4742-8349-1028710992a0/9e673ea1-d5ae-4157-89d9-c50410c687a1"
+          (reference "U3") (unit 1)
+        )
+      )
+    )
+  )
+  (symbol (lib_id "power:+3V3") (at 123.19 78.74 0) (unit 1)
+    (in_bom yes) (on_board yes) (dnp no) (fields_autoplaced)
+    (property "Reference" "#PWR031" (at 123.19 82.55 0)
+      (effects (font (size 1.27 1.27)) hide)
+    )
+    (property "Value" "+3V3" (at 123.19 73.66 0)
+      (effects (font (size 1.27 1.27)))
+    )
+    (property "Footprint" "" (at 123.19 78.74 0)
+      (effects (font (size 1.27 1.27)) hide)
+    )
+    (property "Datasheet" "" (at 123.19 78.74 0)
+      (effects (font (size 1.27 1.27)) hide)
+    )
+    (pin "1")
+    (instances
+      (project "blmd_hardware"
+        (path "/181c0b55-802a-4742-8349-1028710992a0/9e673ea1-d5ae-4157-89d9-c50410c687a1"
+          (reference "#PWR031") (unit 1)
+        )
+      )
+    )
+  )
+  (symbol (lib_id "Device:C") (at 109.22 78.74 90) (unit 1)
+    (in_bom yes) (on_board yes) (dnp no) (fields_autoplaced)
+    (property "Reference" "C24" (at 109.22 71.12 90)
+      (effects (font (size 1.27 1.27)))
+    )
+    (property "Value" "100n" (at 109.22 73.66 90)
+      (effects (font (size 1.27 1.27)))
+    )
+    (property "Footprint" "" (at 113.03 77.7748 0)
+      (effects (font (size 1.27 1.27)) hide)
+    )
+    (property "Datasheet" "~" (at 109.22 78.74 0)
+      (effects (font (size 1.27 1.27)) hide)
+    )
+    (pin "1")
+    (pin "2")
+    (instances
+      (project "blmd_hardware"
+        (path "/181c0b55-802a-4742-8349-1028710992a0/9e673ea1-d5ae-4157-89d9-c50410c687a1"
+          (reference "C24") (unit 1)
+        )
+      )
+    )
+  )
 )

Commit message: 部品配置完了(暫定)
Parts:
- C24: footprint (none) -> Capacitor_SMD:C_0603_1608Metric_Pad1.08x0.95mm_HandSolder
- U3: footprint digikey-footprints:SOIC-8_W3.9mm -> Package_SO:SOIC-8_3.9x4.9mm_P1.27mm
Changed lines of the file:
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@@
       (effects (font (size 1.524 1.524)) (justify left))
     )
-    (property "Footprint" "digikey-footprints:SOIC-8_W3.9mm" (at 125.73 76.2 0)
+    (property "Footprint" "Package_SO:SOIC-8_3.9x4.9mm_P1.27mm" (at 125.73 76.2 0)
       (effects (font (size 1.524 1.524)) (justify left) hide)
     )
@@
       (effects (font (size 1.27 1.27)))
     )
-    (property "Footprint" "" (at 113.03 77.7748 0)
+    (property "Footprint" "Capacitor_SMD:C_0603_1608Metric_Pad1.08x0.95mm_HandSolder" (at 113.03 77.7748 0)
       (effects (font (size 1.27 1.27)) hide)
     )
